Commit message: 修复：arm-only 时通过 use_gripper 禁用 Robotiq URDF/SRDF

File: robots/fr3/fr3_robotiq.srdf.xacro (robot description, xacro)
@@ -8,4 +8,5 @@
   <xacro:arg name="hand" default="false" />
   <xacro:arg name="ee_id" default="robotiq_gripper" />
+  <xacro:arg name="use_gripper" default="true" />
   <xacro:franka_arm_srdf arm_id="$(arg arm_id)"
                       hand="$(arg hand)"
@@ -14,35 +15,37 @@
                       arm_prefix= "$(arg arm_prefix)">
   </xacro:franka_arm_srdf>
-  <group name="gripper">
-    <joint name="robotiq_85_left_knuckle_joint" />
-    <joint name="robotiq_85_right_knuckle_joint" />
-    <joint name="robotiq_85_left_inner_knuckle_joint" />
-    <joint name="robotiq_85_right_inner_knuckle_joint" />
-    <joint name="robotiq_85_left_finger_tip_joint" />
-    <joint name="robotiq_85_right_finger_tip_joint" />
-  </group>
-  <end_effector name="robotiq_gripper" parent_link="fr3_link8" group="gripper" parent_group="fr3_arm" />
-  <disable_collisions link1="robotiq_85_base_link" link2="robotiq_85_left_knuckle_link" reason="Adjacent" />
-  <disable_collisions link1="robotiq_85_base_link" link2="robotiq_85_right_knuckle_link" reason="Adjacent" />
-  <disable_collisions link1="robotiq_85_base_link" link2="robotiq_85_left_inner_knuckle_link" reason="Adjacent" />
-  <disable_collisions link1="robotiq_85_base_link" link2="robotiq_85_right_inner_knuckle_link" reason="Adjacent" />
-  <disable_collisions link1="robotiq_85_left_knuckle_link" link2="robotiq_85_left_finger_link" reason="Adjacent" />
-  <disable_collisions link1="robotiq_85_right_knuckle_link" link2="robotiq_85_right_finger_link" reason="Adjacent" />
-  <disable_collisions link1="robotiq_85_left_finger_link" link2="robotiq_85_left_finger_tip_link" reason="Adjacent" />
-  <disable_collisions link1="robotiq_85_right_finger_link" link2="robotiq_85_right_finger_tip_link" reason="Adjacent" />
-  <disable_collisions link1="robotiq_85_left_inner_knuckle_link" link2="robotiq_85_left_finger_link" reason="Never" />
-  <disable_collisions link1="robotiq_85_right_inner_knuckle_link" link2="robotiq_85_right_finger_link" reason="Never" />
-  <disable_collisions link1="robotiq_85_left_knuckle_link" link2="robotiq_85_left_inner_knuckle_link" reason="Never" />
-  <disable_collisions link1="robotiq_85_right_knuckle_link" link2="robotiq_85_right_inner_knuckle_link" reason="Never" />
-  <disable_collisions link1="robotiq_85_left_finger_tip_link" link2="robotiq_85_right_finger_tip_link" reason="Never" />
-  <disable_collisions link1="robotiq_85_left_finger_link" link2="robotiq_85_right_finger_link" reason="Never" />
-  <disable_collisions link1="robotiq_85_left_knuckle_link" link2="robotiq_85_right_knuckle_link" reason="Never" />
-  <!-- 忽略右指尖和右内关节的碰撞 -->
-<disable_collisions link1="robotiq_85_right_finger_tip_link" link2="robotiq_85_right_inner_knuckle_link" reason="Default" />
-<!-- 通常为了保险，左边的也加上 -->
-<disable_collisions link1="robotiq_85_left_finger_tip_link" link2="robotiq_85_left_inner_knuckle_link" reason="Default" />
-  <disable_collisions link1="fr3_link8" link2="robotiq_85_base_link" reason="Adjacent" />
-  <disable_collisions link1="fr3_link7" link2="robotiq_85_base_link" reason="Default" />
-  <disable_collisions link1="fr3_link7" link2="robotiq_85_left_knuckle_link" reason="Default" />
-  <disable_collisions link1="fr3_link7" link2="robotiq_85_right_knuckle_link" reason="Default" />
+  <xacro:if value="$(arg use_gripper)">
+    <group name="gripper">
+      <joint name="robotiq_85_left_knuckle_joint" />
+      <joint name="robotiq_85_right_knuckle_joint" />
+      <joint name="robotiq_85_left_inner_knuckle_joint" />
+      <joint name="robotiq_85_right_inner_knuckle_joint" />
+      <joint name="robotiq_85_left_finger_tip_joint" />
+      <joint name="robotiq_85_right_finger_tip_joint" />
+    </group>
+    <end_effector name="robotiq_gripper" parent_link="fr3_link8" group="gripper" parent_group="fr3_arm" />
+    <disable_collisions link1="robotiq_85_base_link" link2="robotiq_85_left_knuckle_link" reason="Adjacent" />
+    <disable_collisions link1="robotiq_85_base_link" link2="robotiq_85_right_knuckle_link" reason="Adjacent" />
+    <disable_collisions link1="robotiq_85_base_link" link2="robotiq_85_left_inner_knuckle_link" reason="Adjacent" />
+    <disable_collisions link1="robotiq_85_base_link" link2="robotiq_85_right_inner_knuckle_link" reason="Adjacent" />
+    <disable_collisions link1="robotiq_85_left_knuckle_link" link2="robotiq_85_left_finger_link" reason="Adjacent" />
+    <disable_collisions link1="robotiq_85_right_knuckle_link" link2="robotiq_85_right_finger_link" reason="Adjacent" />
+    <disable_collisions link1="robotiq_85_left_finger_link" link2="robotiq_85_left_finger_tip_link" reason="Adjacent" />
+    <disable_collisions link1="robotiq_85_right_finger_link" link2="robotiq_85_right_finger_tip_link" reason="Adjacent" />
+    <disable_collisions link1="robotiq_85_left_inner_knuckle_link" link2="robotiq_85_left_finger_link" reason="Never" />
+    <disable_collisions link1="robotiq_85_right_inner_knuckle_link" link2="robotiq_85_right_finger_link" reason="Never" />
+    <disable_collisions link1="robotiq_85_left_knuckle_link" link2="robotiq_85_left_inner_knuckle_link" reason="Never" />
+    <disable_collisions link1="robotiq_85_right_knuckle_link" link2="robotiq_85_right_inner_knuckle_link" reason="Never" />
+    <disable_collisions link1="robotiq_85_left_finger_tip_link" link2="robotiq_85_right_finger_tip_link" reason="Never" />
+    <disable_collisions link1="robotiq_85_left_finger_link" link2="robotiq_85_right_finger_link" reason="Never" />
+    <disable_collisions link1="robotiq_85_left_knuckle_link" link2="robotiq_85_right_knuckle_link" reason="Never" />
+    <!-- 忽略右指尖和右内关节的碰撞 -->
+    <disable_collisions link1="robotiq_85_right_finger_tip_link" link2="robotiq_85_right_inner_knuckle_link" reason="Default" />
+    <!-- 通常为了保险，左边的也加上 -->
+    <disable_collisions link1="robotiq_85_left_finger_tip_link" link2="robotiq_85_left_inner_knuckle_link" reason="Default" />
+    <disable_collisions link1="fr3_link8" link2="robotiq_85_base_link" reason="Adjacent" />
+    <disable_collisions link1="fr3_link7" link2="robotiq_85_base_link" reason="Default" />
+    <disable_collisions link1="fr3_link7" link2="robotiq_85_left_knuckle_link" reason="Default" />
+    <disable_collisions link1="fr3_link7" link2="robotiq_85_right_knuckle_link" reason="Default" />
+  </xacro:if>
 </robot>
